File: KDT_Hierarchical_KiBot.kicad_pcb (KiCad board)
At the start: 2 copper layers, 0 parts

Commit message: QR Code Added
Parts:
- added QR1: QR_Revision, ProjectQR:QR_Revision, F.Cu at (201.2, 76.9)
