File: KDT_Hierarchical_KiBot.kicad_pcb (KiCad board)
At the start: 4 copper layers, 0 parts

Commit message: QR Code Added
Parts:
- added QR1: QR_Revision, ProjectQR:QR_Revision, F.Cu at (165.7, 67.9)
